File: usb hub.kicad_pcb (KiCad board)
At the start: 2 copper layers, 22 parts, among them J1 TYPE_C, U1 FE1.1s

Commit message: all routes fixed AND placed parts
Parts:
- moved C1 45.4 mm to (125.2, 97.8)
- moved C2 43.3 mm to (127.3, 100.2)
- moved C3 32.5 mm to (144.7, 99.8)
- moved C5 27.3 mm to (172.7, 98.8)
- moved C4 25.4 mm to (158.6, 98.8)
- moved R1 2.83 mm to (125.2, 98.6), turned to 0 degrees
Connections:
- J1 pad A1: (no net) -> GNDREF
- J1 pad A12: (no net) -> GNDREF
- J1 pad A4: (no net) -> +5V
- J1 pad A9: (no net) -> +5V
- J1 pad B1: (no net) -> GNDREF
- J1 pad B12: (no net) -> GNDREF
- J1 pad B4: (no net) -> +5V
- J1 pad B9: (no net) -> +5V
Routing:
- net GNDREF: track 2.40 -> 8.01 mm
- net +5V: track 0.00 -> 4.85 mm
- net Net-(J1-CC2): track 4.28 -> 0.00 mm
- net (no net): track 1.60 -> 0.00 mm
Changed lines of the file:
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@@
 	(footprint "Resistor_SMD:R_01005_0402Metric"
 		(layer "F.Cu")
-		(at 127.2 96.6 180)
+		(at 125.2 98.6)
 		(descr "Resistor SMD 01005 (0402 Metric), square (rectangular) end terminal, IPC_7351 nominal, (Body size source: http://www.vishay.com/docs/20056/crcw01005e3.pdf), generated with kicad-footprint-generator")
 		(tags "resistor")
@@
 			(at 0 -1 360)
 			(layer "F.SilkS")
+			(hide yes)
 			(effects
 				(font
@@
 		)
 		(property "Footprint" "Resistor_SMD:R_01005_0402Metric"
-			(at 0 0 180)
+			(at 0 0 0)
 			(unlocked yes)
 			(layer "F.Fab")
@@
 		)
 		(property "Datasheet" ""
-			(at 0 0 180)
+			(at 0 0 0)
 			(unlocked yes)
 			(layer "F.Fab")
@@
 		)
 		(property "Description" "Resistor"
-			(at 0 0 180)
+			(at 0 0 0)
 			(unlocked yes)
 			(layer "F.Fab")
@@
 		(attr smd)
 		(fp_line
-			(start 0.6 0.3)
-			(end -0.6 0.3)
+			(start -0.6 -0.3)
+			(end 0.6 -0.3)
 			(stroke
 				(width 0.05)
@@
 		)
 		(fp_line
-			(start 0.6 -0.3)
-			(end 0.6 0.3)
+			(start -0.6 0.3)
+			(end -0.6 -0.3)
 			(stroke
 				(width 0.05)
@@
 		)
 		(fp_line
-			(start -0.6 0.3)
-			(end -0.6 -0.3)
+			(start 0.6 -0.3)
+			(end 0.6 0.3)
 			(stroke
 				(width 0.05)
@@
 		)
 		(fp_line
-			(start -0.6 -0.3)
-			(end 0.6 -0.3)
+			(start 0.6 0.3)
+			(end -0.6 0.3)
 			(stroke
 				(width 0.05)
@@
 		)
 		(fp_line
-			(start 0.2 0.1)
-			(end -0.2 0.1)
+			(start -0.2 -0.1)
+			(end 0.2 -0.1)
 			(stroke
 				(width 0.1)
@@
 		)
 		(fp_line
-			(start 0.2 -0.1)
-			(end 0.2 0.1)
+			(start -0.2 0.1)
+			(end -0.2 -0.1)
 			(stroke
 				(width 0.1)
@@
 		)
 		(fp_line
-			(start -0.2 0.1)
-			(end -0.2 -0.1)
+			(start 0.2 -0.1)
+			(end 0.2 0.1)
 			(stroke
 				(width 0.1)
@@
 		)
 		(fp_line
-			(start -0.2 -0.1)
-			(end 0.2 -0.1)
+			(start 0.2 0.1)
+			(end -0.2 0.1)
 			(stroke
 				(width 0.1)
@@
 		)
 		(fp_text user "${REFERENCE}"
-			(at 0 -0.62 360)
-			(layer "F.Fab")
+			(at 1 0 0)
+			(layer "F.SilkS")
 			(effects
 				(font
@@
 		)
 		(pad "" smd roundrect
-			(at -0.275 0 180)
+			(at -0.275 0)
 			(size 0.27 0.27)
 			(layers "F.Paste")
@@
 		)
 		(pad "" smd roundrect
-			(at 0.275 0 180)
+			(at 0.275 0)
 			(size 0.27 0.27)
 			(layers "F.Paste")
@@
 		)
 		(pad "1" smd roundrect
-			(at -0.25 0 180)
+			(at -0.25 0)
 			(size 0.4 0.3)
 			(layers "F.Cu" "F.Mask")
@@
 		)
 		(pad "2" smd roundrect
-			(at 0.25 0 180)
+			(at 0.25 0)
 			(size 0.4 0.3)
 			(layers "F.Cu" "F.Mask")
@@
 	(footprint "Capacitor_SMD:C_0201_0603Metric"
 		(layer "F.Cu")
-		(at 162.755 126.8)
+		(at 144.745 99.8)
 		(descr "Capacitor SMD 0201 (0603 Metric), square (rectangular) end terminal, IPC_7351 nominal, (Body size source: https://www.vishay.com/docs/20052/crcw0201e3.pdf), generated with kicad-footprint-generator")
 		(tags "capacitor")
@@
 	(footprint "Capacitor_SMD:C_0201_0603Metric"
 		(layer "F.Cu")
-		(at 165.205 123.3)
+		(at 158.6 98.8)
 		(descr "Capacitor SMD 0201 (0603 Metric), square (rectangular) end terminal, IPC_7351 nominal, (Body size source: https://www.vishay.com/docs/20052/crcw0201e3.pdf), generated with kicad-footprint-generator")
 		(tags "capacitor")
@@
 	(footprint "Capacitor_SMD:C_0201_0603Metric"
 		(layer "F.Cu")
-		(at 162.755 123.3)
+		(at 125.2 97.8)
 		(descr "Capacitor SMD 0201 (0603 Metric), square (rectangular) end terminal, IPC_7351 nominal, (Body size source: https://www.vishay.com/docs/20052/crcw0201e3.pdf), generated with kicad-footprint-generator")
 		(tags "capacitor")
@@
 			(at 0 -1.05 0)
 			(layer "F.SilkS")
+			(hide yes)
 			(effects
 				(font
@@
 			(at 0 1.05 0)
 			(layer "F.Fab")
+			(hide yes)
 			(effects
 				(font
@@
 		)
 		(fp_text user "${REFERENCE}"
-			(at 0 -0.68 0)
-			(layer "F.Fab")
+			(at 1 0 0)
+			(layer "F.SilkS")
 			(effects
 				(font
@@
 			(size 0.6 1.45)
 			(layers "F.Cu" "F.Paste" "F.Mask")
+			(net 21 "GNDREF")
+			(pinfunction "GND")
+			(pintype "power_in")
 		)
 		(pad "A4" smd rect
@@
 			(size 0.6 1.45)
 			(layers "F.Cu" "F.Paste" "F.Mask")
+			(net 14 "+5V")
+			(pinfunction "VBUS")
+			(pintype "power_in")
 		)
 		(pad "A5" smd rect
@@
 			(size 0.6 1.45)
 			(layers "F.Cu" "F.Paste" "F.Mask")
+			(net 14 "+5V")
+			(pinfunction "VBUS")
+			(pintype "power_in")
 		)
 		(pad "A12" smd rect
@@
 			(size 0.6 1.45)
 			(layers "F.Cu" "F.Paste" "F.Mask")
+			(net 21 "GNDREF")
+			(pinfunction "GND")
+			(pintype "power_in")
 		)
 		(pad "B1" smd rect
@@
 			(size 0.6 1.45)
 			(layers "F.Cu" "F.Paste" "F.Mask")
+			(net 21 "GNDREF")
+			(pinfunction "GND")
+			(pintype "power_in")
 		)
 		(pad "B4" smd rect
@@
 			(size 0.6 1.45)
 			(layers "F.Cu" "F.Paste" "F.Mask")
+			(net 14 "+5V")
+			(pinfunction "VBUS")
+			(pintype "power_in")
 		)
 		(pad "B5" smd rect
@@
 			(size 0.6 1.45)
 			(layers "F.Cu" "F.Paste" "F.Mask")
+			(net 14 "+5V")
+			(pinfunction "VBUS")
+			(pintype "power_in")
 		)
 		(pad "B12" smd rect
@@
 			(size 0.6 1.45)
 			(layers "F.Cu" "F.Paste" "F.Mask")
+			(net 21 "GNDREF")
+			(pinfunction "GND")
+			(pintype "power_in")
 		)
 		(pad "S1" thru_hole oval
@@
 	(footprint "Capacitor_SMD:C_0201_0603Metric"
 		(layer "F.Cu")
-		(at 162.755 125.05)
+		(at 127.345 100.2)
 		(descr "Capacitor SMD 0201 (0603 Metric), square (rectangular) end terminal, IPC_7351 nominal, (Body size source: https://www.vishay.com/docs/20052/crcw0201e3.pdf), generated with kicad-footprint-generator")
 		(tags "capacitor")
@@
 	(footprint "Capacitor_SMD:C_0201_0603Metric"
 		(layer "F.Cu")
-		(at 165.205 125.05)
+		(at 172.655 98.8)
 		(descr "Capacitor SMD 0201 (0603 Metric), square (rectangular) end terminal, IPC_7351 nominal, (Body size source: https://www.vishay.com/docs/20052/crcw0201e3.pdf), generated with kicad-footprint-generator")
 		(tags "capacitor")
@@
 	)
 	(segment
-		(start 125.295 89.35)
-		(end 125.295 88.55)
+		(start 126.22 94.25)
+		(end 125.295 94.25)
 		(width 0.2)
 		(layer "F.Cu")
-		(net 0)
+		(net 14)
 	)
 	(segment
-		(start 125.295 94.25)
-		(end 125.295 95.05)
+		(start 126.32 97)
+		(end 126.32 94.35)
+		(width 0.2)
+		(layer "F.Cu")
+		(net 14)
+	)
+	(segment
+		(start 126.32 94.35)
+		(end 126.22 94.25)
+		(width 0.2)
+		(layer "F.Cu")
+		(net 14)
+	)
+	(segment
+		(start 125.52 97.8)
+		(end 126.32 97)
 		(width 0.2)
 		(layer "F.Cu")
-		(net 0)
+		(net 14)
 	)
 	(segment
@@
 	)
 	(segment
-		(start 126.95 94.28)
-		(end 126.22 93.55)
+		(start 124.38 96.12)
+		(end 124.38 95.965002)
 		(width 0.2)
 		(layer "F.Cu")
-		(net 24)
+		(net 21)
 	)
 	(segment
-		(start 126.95 96.6)
-		(end 126.95 94.28)
+		(start 125.295 95.050002)
+		(end 125.295 95.05)
 		(width 0.2)
 		(layer "F.Cu")
-		(net 24)
+		(net 21)
 	)
 	(segment
-		(start 126.22 93.55)
-		(end 125.295 93.55)
+		(start 124.95 98.6)
+		(end 124.95 97.87)
 		(width 0.2)
 		(layer "F.Cu")
-		(net 24)
+		(net 21)
+	)
+	(segment
+		(start 124.88 96.62)
+		(end 124.38 96.12)
+		(width 0.2)
+		(layer "F.Cu")
+		(net 21)
+	)
+	(segment
+		(start 125.295 88.55)
+		(end 125.295 88.395)
+		(width 0.2)
+		(layer "F.Cu")
+		(net 21)
+	)
+	(segment
+		(start 125.295 88.395)
+		(end 124.38 87.48)
+		(width 0.2)
+		(layer "F.Cu")
+		(net 21)
+	)
+	(segment
+		(start 124.95 97.87)
+		(end 124.88 97.8)
+		(width 0.2)
+		(layer "F.Cu")
+		(net 21)
+	)
+	(segment
+		(start 124.88 97.8)
+		(end 124.88 96.62)
+		(width 0.2)
+		(layer "F.Cu")
+		(net 21)
+	)
+	(segment
+		(start 124.38 95.965002)
+		(end 125.295 95.050002)
+		(width 0.2)
+		(layer "F.Cu")
+		(net 21)
 	)
 	(segment

Commit message: bit of routing
Parts:
- moved C5 33.3 mm to (139.4, 99.1), turned to 90 degrees
- moved C4 12.2 mm to (170.6, 100.8)
- moved C2 10.2 mm to (137.5, 100.8)
- moved C3 9.29 mm to (154.0, 100.6)
- moved R1 5.39 mm to (127.2, 93.6), turned to 180 degrees
- moved C1 5.28 mm to (121.0, 101.0)
- moved R2 3.81 mm to (127.2, 90.6), turned to 180 degrees
- moved R3 2.48 mm to (137.6, 89.6)
- moved R6 0.80 mm to (140.7, 99.1)
- moved U1 0.80 mm to (136.6, 94.8)
- moved PWR1 0.80 mm to (137.6, 88.0), turned to -90 degrees
- moved R4 0.80 mm to (136.6, 89.6)
- moved R5 0.80 mm to (134.2, 89.6)
- moved USB_1 0.80 mm to (136.6, 88.0)
- moved USB_2 0.80 mm to (135.8, 88.0)
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Connections:
- PWR1 pad 1: Net-(PWR1-K) -> GNDREF
- R3 pad 1: GNDREF -> Net-(PWR1-A)
- R3 pad 2: Net-(PWR1-K) -> Net-(U1-DRV)
- U1 pad 22: Net-(PWR1-A) -> Net-(U1-DRV)
Routing:
- net +5V: track 4.85 -> 93.2 mm
- net +3.3V: track 0.00 -> 10.7 mm
- net GNDREF: track 8.01 -> 3.57 mm, vias 0 -> 1
- net Net-(J1-CC1): track 5.33 -> 1.68 mm
- net USB_DM: track 0.00 -> 3.05 mm
- net USB_DP: track 0.00 -> 2.98 mm
- net Net-(U1-DRV): track 0.00 -> 2.83 mm
- net Net-(U1-LED1/EESCL): track 0.00 -> 2.68 mm
- net Net-(U1-LED2): track 0.00 -> 2.62 mm
- net Net-(J1-CC2): track 0.00 -> 1.68 mm
- net Net-(U1-REXT): track 1.43 -> 0.00 mm
- net Net-(PWR1-A): track 0.00 -> 0.91 mm
- net Net-(PWR1-K): track 0.80 -> 0.00 mm
- added copper zone on B.Cu, net GNDREF
- added copper zone on F.Cu, net GNDREF
Other:
- board outline added: 65 x 30.4 mm

Commit message: ITS FINISHED!!!
Parts:
- moved R6 0.14 mm to (140.7, 99.0)
Connections:
- C5 pad 2: Net-(U1-VD18) -> Net-(U1-VD18_O)
- U1 pad 12: Net-(U1-VD18) -> Net-(U1-VD18_O)
- U1 pad 28: Net-(U1-VD18) -> unconnected-(U1-VD18-Pad28)
Routing:
- net D4_P: track 0.00 -> 46.0 mm, vias 0 -> 2
- net D4_N: track 0.00 -> 45.2 mm, vias 0 -> 2
- net D3_P: track 0.00 -> 27.3 mm, vias 0 -> 2
- net D3_N: track 0.00 -> 27.2 mm, vias 0 -> 2
- net USB_DM: track 3.05 -> 22.7 mm, vias 0 -> 2
- net D1_N: track 0.00 -> 17.4 mm, vias 0 -> 2
- net USB_DP: track 2.98 -> 19.6 mm, vias 0 -> 2
- net D1_P: track 0.00 -> 16.0 mm, vias 0 -> 2
- net D2_P: track 0.00 -> 10.2 mm, vias 0 -> 2
- net D2_N: track 0.00 -> 9.74 mm, vias 0 -> 2
- net +5V: track 93.2 -> 101.2 mm
- net GNDREF: track 3.57 -> 0.98 mm, vias 1 -> 3
- net +3.3V: track 10.7 -> 12.5 mm
- net Net-(U1-VD18_O): track 0.00 -> 1.36 mm
- net Net-(U1-REXT): track 0.00 -> 1.28 mm
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Other:
- outline, holes or cut-outs redrawn
